File: kicad/vue2.kicad_sch (KiCad schematic)
At the start: 26 parts, among them J1 Conn_01x07_Male, U5 ESP32-S2-WROVER

Commit message: Update schematic
As described in https://github.com/emporia-vue-local/esphome/discussions/173#discussioncomment-6137086

Thank you @g3gg0!

Also this ends up upgrading the project to Kicad 7
Parts:
- removed U5: ESP32-S2-WROVER, RF_Module:ESP32-S2-WROVER, symbol RF_Module:ESP32-S2-WROVER
- added U5: ESP32-WROVER-IB, RF_Module:ESP32-WROOM-32, symbol RF_Module:ESP32-WROOM-32
Connections:
- net +3V3: now also R43.1, R44.2, U5.2 (VDD)
- net EMAC_RXD1: now also U5.11 (IO26)
- net GND: now also C20.2, U5.1 (GND), U5.15 (GND), U5.38 (GND), U5.39 (GND)
- net I2CCLK: now also R44.1, U5.36 (IO22)
- net I2CDAT: now also R43.2, U5.33 (IO21)
- net IO0: now also U5.25 (IO0)
- net RXD: now also U5.34 (RXD0/IO3)
- net TXD: now also U5.35 (TXD0/IO1)
- net at R115.2, R119.1: now also U5.7 (IO35)
- net BUZ+: now reaches R143.2, SP1.1 (-)
- net BUZ+: now also U5.14 (IO12)
- net at R114.1, R118.1: now also U5.6 (IO34)
- net at R113.2, R117.1: now also U5.9 (IO33)
- net at R112.2, R116.2: now also U5.8 (IO32)
- net BUZ renamed BUZ-
- net BUZ-: now also U5.12 (IO27)
- net EN renamed ESP_EN
- net ESP_EN: now also U5.3 (EN)
- new net SWCLK: U5.13 (IO14)
- new net SWDIO: U5.16 (IO13)
- new net ~{AT_RST}: U5.26 (IO4)
- no-connect marks 0 -> 6
Other:
- sheet ADC ports: added none; removed MTCK, MTMS
- moved on the sheet: C18, C19, C20, R112, R113, R114, R115, R116, R117, R118, R119, R143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
